File: noncontact-electrodes/noncontact-electrodes.kicad_pcb (KiCad board)
At the start: 2 copper layers, 25.1 x 25 mm, 13 parts, among them P1 CONN_1, P2 CONN_1, P3 CONN_1, P4 CONN_1, P5 CONN_1, P6 CONN_1, U1 TLC272

Commit message: fixed diodes on amplifier pcb
Parts:
- U1: value TLC272 -> lmp7702
Changed lines of the file:
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@@
     (links 16)
     (no_connects 0)
-    (area 0 0 0 0)
+    (area 11.887999 11.887999 38.033586 37.007001)
     (thickness 1.6)
     (drawings 4)
@@
       (effects (font (size 1.143 1.143) (thickness 0.1524)))
     )
-    (fp_text value TLC272 (at 0 1.016 270) (layer F.SilkS)
+    (fp_text value lmp7702 (at 0 1.016 270) (layer F.SilkS)
       (effects (font (size 0.889 0.889) (thickness 0.1524)))
     )

Commit message: added discontinued notice
Changed lines of the file:
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@@
   (general
     (links 16)
-    (no_connects 0)
+    (no_connects 1)
     (area 11.887999 11.887999 38.033586 37.007001)
     (thickness 1.6)
@@
     (descr "module 1 pin (ou trou mecanique de percage)")
     (tags DEV)
-    (fp_text reference P3 (at 0 -3.50012) (layer F.SilkS)
+    (fp_text reference P3 (at -0.254 -0.1905) (layer F.SilkS)
       (effects (font (size 0.5 0.5) (thickness 0.1)))
     )
@@
     (descr "module 1 pin (ou trou mecanique de percage)")
     (tags DEV)
-    (fp_text reference P5 (at 0 -3.50012) (layer F.SilkS)
+    (fp_text reference P5 (at -0.1016 -0.5969) (layer F.SilkS)
       (effects (font (size 0.5 0.5) (thickness 0.1)))
     )
@@
     (descr "module 1 pin (ou trou mecanique de percage)")
     (tags DEV)
-    (fp_text reference P6 (at 0 -3.50012) (layer F.SilkS)
+    (fp_text reference P6 (at -0.8636 -0.1397) (layer F.SilkS)
       (effects (font (size 0.5 0.5) (thickness 0.1)))
     )
@@
     (descr "module 1 pin (ou trou mecanique de percage)")
     (tags DEV)
-    (fp_text reference P4 (at 0 -3.50012) (layer F.SilkS)
+    (fp_text reference P4 (at -0.1016 0.1524) (layer F.SilkS)
       (effects (font (size 0.5 0.5) (thickness 0.1)))
     )
@@
   (segment (start 30.2895 21.209) (end 35.433 21.209) (width 0.5) (layer F.Cu) (net 5))
   (segment (start 35.433 21.209) (end 35.814 21.59) (width 0.5) (layer F.Cu) (net 5))
-  (segment (start 30.2895 18.4785) (end 35.814 18.4785) (width 0.5) (layer F.Cu) (net 6))
+  (segment (start 30.2895 18.4785) (end 35.814 18.4785) (width 0.5) (layer F.Cu) (net 6) (status 20))
   (segment (start 24.257 26.797) (end 21.0185 26.797) (width 0.5) (layer F.Cu) (net 7))
   (segment (start 21.0185 20.3835) (end 24.1935 20.3835) (width 0.5) (layer F.Cu) (net 8))
